File: power.kicad_sch (KiCad schematic)
At the start: 54 parts, among them J3 Conn_01x02, J4 Conn_01x02, Q6 Si2302, Q7 Si2302, Q8 Q_PMOS_GSD, U1 TP4056, U16 PS7516, U2 SGM2039, U6 SGM2033-1.8, U8 SGM8040-1

Commit message: 修复R12封装错误，1210电容改为1206电阻
Parts:
- R12: footprint Capacitor_SMD:C_1210_3225Metric -> Resistor_SMD:R_1206_3216Metric
Changed lines of the file:
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@@
 			)
 		)
-		(property "Footprint" "Capacitor_SMD:C_1210_3225Metric"
+		(property "Footprint" "Resistor_SMD:R_1206_3216Metric"
 			(at 132.08 55.372 90)
 			(effects
